Commit message: correction with z axis

File: ros_ws/src/pekauto_task/model/model1.urdf (robot description, URDF)
Before this commit: robot model, 3 links, 2 joints
Links:
- added link left_front_l; collision cylinder length=0.2 radius=0.2; visual cylinder length=0.2 radius=0.2
- added link left_rear_l; collision cylinder length=0.2 radius=0.2; visual cylinder length=0.2 radius=0.2
- added link right_front_l; collision cylinder length=0.2 radius=0.2; visual cylinder length=0.2 radius=0.2
- added link right_rear_l; collision cylinder length=0.2 radius=0.2; visual cylinder length=0.2 radius=0.2
Joints:
- added joint left_front: type fixed, parent base_link, child left_front_l, origin xyz=1 0.75 0 rpy=0 0 0
- added joint left_rear: type fixed, parent base_link, child left_rear_l, origin xyz=-1 0.75 0 rpy=0 0 0
- added joint right_front: type fixed, parent base_link, child right_front_l, origin xyz=1 -0.75 0 rpy=0 0 0
- added joint right_rear: type fixed, parent base_link, child right_rear_l, origin xyz=-1 -0.75 0 rpy=0 0 0
